File: hardware/ludusProtoShield.brd (EAGLE design)
At the start: 59.7 x 53.3 mm, 54 parts, among them U1 ARDUINO, U3 TB6612FNG

Commit message: Updated design to resolve all issues
Parts:
- removed FRAME1: FRAME-LETTER, SparkFun-Aesthetics:CREATIVE_COMMONS
- removed SJ1, SJ2: JUMPER-PAD-3-2OF3_NC_BY_PASTE, SparkFun-Passives:PAD-JUMPER-3-2OF3_NC_BY_PASTE_YES_SILK_FULL_BOX
- added FRAME2: FRAME-LEDGER, SparkFun-Aesthetics:CREATIVE_COMMONS
- added S1, S2: (no value), SparkFun-Electromechanical:AYZ0202
- U$1: value SFE_LUDUS -> SFE_LUDUSSFE_LUDUS-M
- moved U$1 6.63 mm to (41.3, 26.7), flipped to the bottom, turned to 270 degrees
Connections:
- net N$20 renamed BIN2
- net ANALOG_PWR_RAIL: now also S1.2; no longer SJ2.2
- net FUSED_VCC: now also S1.3, S2.3; no longer SJ1.3, SJ2.3
- net FUSED_VIN: now also S1.1, S2.1; no longer SJ1.1, SJ2.1
- net PWR_RAIL: now also S2.2; no longer SJ1.2
Routing:
- net N$21: track 0.00 -> 5.84 mm
- net N$20: track 0.00 -> 5.21 mm
- net N$43: track 0.00 -> 4.95 mm
- net N$22: track 0.00 -> 4.95 mm
- net FUSED_VIN: track 82.8 -> 86.2 mm, vias 4 -> 6
- net PWR_RAIL: track 42.6 -> 45.9 mm
- net FUSED_VCC: track 72.0 -> 71.6 mm, vias 2 -> 3
Other:
- board text added: "V02"
- board text removed: "POWER SEL"
- board text removed: "V11"
